File: 01_sheet/PICO_SDR.brd (EAGLE design)
At the start: 98.7 x 64.8 mm, 70 parts, among them IC2 MCP6022, J1 DCJ0202, J2 FC68131, J3 FC68133, SW1 EC12E_SW, U2 74CBTLV3253, U3 PAM8403DR

Commit message: sheet
Parts:
- added JP3: Speaker, pinhead:1X02
- added U$10, U$8, U$9: (no value), special:DRIL-2,5
- C11, C12, C13, C19, C2, C26, C27, C28, C29, C3, C6, C7: device rcl:C1206 -> rcl:C0805
- C14, C32: value (none) -> 100n
- C15, C16, C17, C20: value (none) -> 100µ; device rcl:E2,5-6E -> rcl:SMC_D
- C18: value (none) -> 470n
- C21: value (none) -> 1µ
- C22: value (none) -> 470n; device rcl:C1206 -> rcl:C0805
- L1, L2: value (none) -> VK200
- R1: value (none) -> 100
- R2: value (none) -> 20k
- R3: value RK09K1130A6S -> 10k
- moved C33 472.6 mm to (58.4, 55.9), flipped to the bottom, turned to 270 degrees
- moved JP1 461.9 mm to (16.5, 59.7)
- moved JP2 461.5 mm to (6.35, 59.7)
- moved SJ4 422.9 mm to (43.2, 55.9), turned to 180 degrees
- moved SJ3 420.5 mm to (43.2, 58.4), turned to 180 degrees
- moved SJ1 413.3 mm to (43.2, 61.0), turned to 180 degrees
- moved C32 413.1 mm to (3.81, 25.4)
- moved SJ2 410.9 mm to (43.2, 53.3), turned to 180 degrees
- moved C29 408.1 mm to (88.9, 62.2), flipped to the bottom
- moved C28 401.4 mm to (83.8, 62.2), flipped to the bottom
- moved C27 393.7 mm to (76.2, 62.2), flipped to the bottom, turned to 180 degrees
- moved C30 387.5 mm to (88.9, 25.4), flipped to the bottom, turned to 270 degrees
- moved C26 387.1 mm to (71.1, 62.2), flipped to the bottom, turned to 180 degrees
- moved C31 382.9 mm to (83.8, 16.5), flipped to the bottom, turned to 270 degrees
- moved L6 382.4 mm to (82.5, 57.1), flipped to the bottom, turned to 270 degrees
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Connections:
- new net N$26: C10.1, C12.2, L3.2
- new net N$27: C5.1, C6.2, L5.2
- net LP+: now also JP3.2
- net LP-: now also JP3.1
- net P_180: no longer C10.1, C12.2, L3.2
- net P_270: no longer C5.1, C6.2, L5.2
Routing:
- net GND: track 0.00 -> 36.4 mm
- net LP-: track 0.00 -> 31.1 mm
- net LP+: track 0.00 -> 26.1 mm
- net N$23: track 0.00 -> 9.08 mm
- net N$3: track 0.00 -> 6.07 mm
- net N$27: track 0.00 -> 6.07 mm
- net N$26: track 0.00 -> 6.07 mm
- net N$20: track 0.00 -> 6.07 mm
- net N$24: track 0.00 -> 4.75 mm
- net P_90: track 0.00 -> 3.26 mm
- net P_270: track 0.00 -> 3.26 mm
- net P_0: track 0.00 -> 3.26 mm
- net P_180: track 0.00 -> 3.26 mm
- net N$6: track 0.00 -> 2.73 mm
- net N$19: track 0.00 -> 2.73 mm
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Other:
- board size 98.7 x 64.8 mm -> 100 x 65 mm

Commit message: new version
Parts:
- removed U$3: RP2350 - Stamp, rp2xxx_stamp:RP2XXX_STAMP_TH
- removed U3: PAM8403DR, PAM8403DR:SOIC127P605X150-16N
- added IC1: RP2350 - Stamp, rp2xxx_stamp:RP2XXX_STAMP_SMD
- added J4: FC68133, FC68133:CLIFF_FC68133
- added JP4: RF, pinhead:1X02
- added U1: 74CBTLV3253, FST3253MX:SOIC127P599X175-16N
- C1: value 220n -> 100n
- C10: value 10µ -> 10n; device rcl:C1206 -> rcl:C0805
- C13: value 100n -> 10n
- C14: value 100n -> 10n; device rcl:C1206 -> rcl:C0805
- C15, C16: value 100µ -> 10n; device rcl:SMC_D -> rcl:C0805
- C17, C20: value 100µ -> 10µ; device rcl:SMC_D -> rcl:C1206
- C18: value 470n -> 10µ
- C19: value 100n -> 10µ; device rcl:C0805 -> rcl:C1206
- C2: value 100n -> 100µ; device rcl:C0805 -> rcl:SMC_D
- C21: value 1µ -> 100µ; device rcl:C1206 -> rcl:SMC_D
- C22: device rcl:C0805 -> rcl:C1206
- C23: value 10µ -> 27p
- C26: value 10n -> 100n
- C27: value 10n -> 27p; device rcl:C0805 -> rcl:C1206
- C28, C29: value 10n -> 10µ; device rcl:C0805 -> rcl:C1206
- C3: value 2,2µ -> 100n; device rcl:C0805 -> rcl:C1206
- C30: value 10µ -> 470n; device rcl:C1206 -> rcl:C0805
- C31: value 10µ -> 100n; device rcl:C1206 -> rcl:C0805
- C32: value 100n -> 100µ; device rcl:C1206 -> rcl:SMC_D
- C33: value 220n -> 1µ
- C4: value 10µ -> 2,2µ; device rcl:C1206 -> rcl:C0805
- C5: value 10µ -> 220n
- C6: value 10n -> 220n; device rcl:C0805 -> rcl:C1206
- C7: value 10n -> 100µ; device rcl:C0805 -> rcl:SMC_D
- C8: value 27p -> 100n; device rcl:C1206 -> rcl:C0805
- C9: value 27p -> 10n; device rcl:C1206 -> rcl:C0805
- J2: value FC68131 -> 629105136821; device FC68131:CLIFF_FC68131 -> Eagle_WR-USB (rev25a):629105136821
- J3: value FC68133 -> FC68131; device FC68133:CLIFF_FC68133 -> FC68131:CLIFF_FC68131
- OLED1: value OLED -> (none)
- R1: value 100 -> 10k
- R12: value 100 -> 10k; device rcl:R0805 -> RK09K1130A6S:RK09K1130A6S
- R13: value 100 -> 20k
- R2: value 20k -> 10k
- R3: value 10k -> 100; device RK09K1130A6S:RK09K1130A6S -> rcl:R0805
- R4, R7: value 100k -> 100
- R5, R6: value 10k -> 100
- R8, R9: value 100 -> 100k
- U2: value 74CBTLV3253 -> PAM8403DR; device FST3253MX:SOIC127P599X175-16N -> PAM8403DR:SOIC127P605X150-16N
- moved J2 91.9 mm to (2.54, 24.1), turned to 270 degrees
- moved C15 71.5 mm to (72.4, 52.1), turned to 180 degrees
- moved C18 69.1 mm to (73.7, 48.3), flipped to the bottom, turned to 270 degrees
- moved C21 68.6 mm to (2.54, 36.8), flipped to the bottom
- moved C17 67.5 mm to (76.2, 48.3), flipped to the bottom, turned to 270 degrees
- moved C32 67.4 mm to (71.1, 29.2), turned to 270 degrees
- moved C14 66.5 mm to (87.6, 52.1), flipped to the bottom
- moved C22 63.9 mm to (20.3, 5.08), flipped to the bottom
- moved C16 61.4 mm to (82.5, 52.1), flipped to the bottom
- moved C2 57.4 mm to (11.4, 20.3)
- moved C1 56.8 mm to (17.8, 19.1), turned to 90 degrees
- moved R12 56.7 mm to (27.0, 15.0), flipped to the top, turned to 0 degrees
- moved R3 56.7 mm to (76.2, 43.2), flipped to the bottom, turned to 90 degrees
- moved R7 56.2 mm to (20.3, 10.2), turned to 90 degrees
- moved R1 53.1 mm to (68.6, 30.5), flipped to the bottom, turned to 0 degrees
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- renumbered U$1 to TR1, U$2 to OLED1
Connections:
- new net D+: IC1.36, J2.3
- new net D-: IC1.35, J2.2
- net +3V3: now also C26.2, C3.2, C7.+, C8.1, R1.2, SJ1.2, SJ2.2, U1.16; no longer C13.2, C14.2, C16.+, C2.1, R6.2, SJ3.2, SJ4.2, U2.16
- net +5V: now also C1.2, C2.+, J2.1; no longer C17.+, C32.2
- net AGND: now also C32.-, C33.1; no longer C20.-, C21.1
- net BAND_0: now also IC1.3; no longer U$3.3, U$3.TH3
- net BAND_1: now also IC1.4; no longer U$3.4, U$3.TH4
- net BAND_2: now also IC1.5; no longer U$3.5, U$3.TH5
- net BIAS: now also C27.2, C4.2, R1.1, R11.1, R2.2, R9.1; no longer C25.2, C3.2, R4.1, R5.2, R6.1, R7.1
- net BUTTON_BACK: now also IC1.18; no longer U$3.18, U$3.TH18
- net BUTTON_FWD: now also IC1.23; no longer U$3.23, U$3.TH23
- net CS: now also IC1.14; no longer U$3.14, U$3.TH14
- net ENCODER_A: now also IC1.22; no longer U$3.22, U$3.TH22
- net ENCODER_B: now also IC1.21; no longer U$3.21, U$3.TH21
- net GND: now also C1.1, C10.1, C15.1, C16.1, C2.-, C22.1, C31.1, C4.1, C7.-, C8.2, C9.1, IC1.31, J2.5, J2.S1, J2.S2, J2.S3, J2.S4, J3.1, R12.E, R2.1, SJ3.2, SJ4.2, U1.1, U1.15, U1.8, U2.11, U2.2; no longer C16.-, C17.-, C18.1, C19.1, C2.2, C27.1, C28.1, C29.1, C32.1, C6.1, C7.1, J2.1, R3.E, R5.1, SJ1.2, SJ2.2, U$3.31, U$3.TH31, U2.1, U2.8, U3.11, U3.15, U3.2
- net LO_I: now also IC1.2, U1.2; no longer U$3.2, U$3.TH2, U2.2
- net LO_Q: now also IC1.1, U1.14; no longer U$3.1, U$3.TH1, U2.14
- net LP+: now also J4.3, J4.4; no longer J3.3, J3.4
- net LP-: now also J4.1, U2.14; no longer J3.1, U3.14
- net MISO: now also IC1.13; no longer U$3.13, U$3.TH13
- net MOSI: now also IC1.16; no longer U$3.16, U$3.TH16
- net N$1: now also IC1.34; no longer U$3.34, U$3.TH34
- net N$10: now also C27.1, R11.2, R6.1; no longer C25.1, R7.2, R9.1
- net N$11: now also C25.1, R5.1; no longer C8.1, R8.1
- net N$12: now also C18.2, R4.2; no longer C4.2, R13.2
- net N$13: now also C23.1, R3.1, R8.2; no longer C9.1, R11.2, R12.1
- net N$14: now also R13.1, U2.10; no longer R2.1, U3.10
- net N$15: now also C17.2, R3.2; no longer C10.2, R12.2
- net N$16: now also R4.1, R9.2; no longer R13.1, R4.2
- net N$17: now also C30.1, R13.2; no longer C22.1, R2.2
- net N$18: now also C5.2; no longer C1.2
- net N$19: now also C20.2, R6.2; no longer C23.2, R9.2
- net N$2: now also C21.-, R7.2; no longer C15.-, R1.2
- net N$20: now also C15.2, C18.1; no longer C11.2, C4.1
- net N$21: now also C28.2, J3.5; no longer C30.2, J2.5
- net N$22: now also C29.2, J3.2; no longer C31.2, J2.2
- net N$23: now also SJ2.1, SJ4.1; no longer SJ1.1, SJ3.1
- net N$24: now also SJ1.1, SJ3.1; no longer SJ2.1, SJ4.1
- net N$25: now also C6.2; no longer C33.2
- net N$26: now also C13.2, C17.1; no longer C10.1, C12.2
- net N$27: now also C14.2, C19.1; no longer C5.1, C6.2
- net N$3: now also C16.2, C20.1; no longer C23.1, C7.2
- net N$4: now also IC1.33; no longer U$3.33, U$3.TH33
- net N$5: now also U1.9; no longer U2.9
- net N$6: now also C19.2, R5.2; no longer C5.2, R8.2
- net N$7: now also U1.7; no longer U2.7
- net N$8: now also C31.2, U2.8; no longer C19.2, U3.8
- net N$9: now also C30.2, R12.S; no longer C22.2, R3.S
- net NF: now also C22.2, R12.A, R7.1; no longer C18.2, R1.1, R3.A
- net OUT_R: now also J4.2, J4.5, U2.16; no longer J3.2, J3.5, U3.16
- net PUSH: now also IC1.6; no longer U$3.6, U$3.TH6
- net P_0: now also C11.2, U1.12, U1.5; no longer C26.2, U2.12, U2.5
- net P_180: now also C9.2, U1.11, U1.4; no longer C27.2, U2.11, U2.4
- net P_270: now also C10.2, U1.10, U1.3; no longer C29.2, U2.10, U2.3
- net P_90: now also C12.2, U1.13, U1.6; no longer C28.2, U2.13, U2.6
- net RF_1: now also C5.1, JP4.2; no longer C1.1
- net RF_2: now also C6.1, JP4.1; no longer C33.1
- net RX_I: now also C23.2, C28.1, IC1.28, R8.1; no longer C30.1, C9.2, R11.1, U$3.28, U$3.TH28
- net RX_Q: now also C25.2, C29.1, IC1.27; no longer C31.1, C8.2, U$3.27, U$3.TH27
- net SCK: now also IC1.15; no longer U$3.15, U$3.TH15
- net SCL: now also IC1.20; no longer U$3.20, U$3.TH20
- net SDA: now also IC1.19; no longer U$3.19, U$3.TH19
- net SPEAKER: now also C21.+, IC1.17; no longer C15.+, U$3.17, U$3.TH17
- net VBAT: now also C32.+, C33.2, IC1.32, U2.12, U2.13, U2.4, U2.5, U2.6; no longer C20.+, C21.2, U$3.32, U$3.TH32, U3.12, U3.13, U3.4, U3.5, U3.6
Routing:
- net GND: track 36.4 -> 448.4 mm, vias 0 -> 3
- net +3V3: track 0.00 -> 195.3 mm, vias 0 -> 4
- net VBAT: track 0.00 -> 107.9 mm, vias 0 -> 2
- net RX_I: track 0.00 -> 91.5 mm, vias 0 -> 5
- net RX_Q: track 0.00 -> 88.0 mm, vias 0 -> 3
- net ENCODER_A: track 0.00 -> 84.7 mm, vias 0 -> 1
- net PUSH: track 0.00 -> 81.9 mm
- net ENCODER_B: track 0.00 -> 72.1 mm, vias 0 -> 2
- net N$9: track 0.00 -> 64.8 mm
- net SDA: track 0.00 -> 55.6 mm, vias 0 -> 2
- net BUTTON_BACK: track 0.00 -> 54.8 mm, vias 0 -> 1
- net SCL: track 0.00 -> 53.9 mm, vias 0 -> 2
- net BUTTON_FWD: track 0.00 -> 53.9 mm, vias 0 -> 1
- net BIAS: track 0.00 -> 50.9 mm, vias 0 -> 1
- net LO_I: track 0.00 -> 50.2 mm, vias 0 -> 1
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- added copper zone on layer 1, net GND
- added copper zone on layer 16, net GND

Commit message: new Version (08.07.25)
Parts:
- removed C32: 100µ, rcl:SMC_D
- removed J2: 629105136821, Eagle_WR-USB (rev25a):629105136821
- removed U2: PAM8403DR, PAM8403DR:SOIC127P605X150-16N
- added FL1, FL2: BLM21SP111SH1D, BLM21SP111SH1D:BEADC2012X105N
- added J5: 629105150521, Eagle_WR-USB (rev25a):629105150521
- added R14: 40k, rcl:R0805
- added R15: 20k, rcl:R0805
- added U3: MAX9716EUAT, MAX9716EUAT:SOP65P490X110-9N
- C31: value 100n -> 1µ
- C6: value 220n -> 100n; device rcl:C1206 -> rcl:C0805
- moved C6 18.7 mm to (40.0, 59.1), flipped to the top, turned to 90 degrees
- moved C33 4.55 mm to (69.2, 32.7), turned to 90 degrees
- moved C2 3.18 mm to (11.4, 17.1)
- moved R13 2.01 mm to (81.9, 27.3)
- moved J1 0.90 mm to (10.8, 13.1)
- moved C8 0.63 mm to (66.0, 38.7)
Connections:
- removed net AGND: C32.-, C33.1
- new net N$28: C6.1, FL1.1, SJ1.2, SJ2.2
- new net N$29: C8.1, FL2.2, U1.16
- net +3V3: now also C33.2, FL1.2, FL2.1, R15.2, U3.6; no longer C8.1, SJ1.2, SJ2.2, U1.16
- net +5V: now also J5.1; no longer J2.1
- net D+: now also J5.3; no longer J2.3
- net D-: now also J5.2; no longer J2.2
- net GND: now also C33.1, C6.2, J5.S1, J5.S2, J5.S3, J5.S4, U3.7, U3.9; no longer J2.5, J2.S1, J2.S2, J2.S3, J2.S4, U2.11, U2.15, U2.2
- net LP-: now also U3.8; no longer U2.14
- net N$14: now also C31.2, U3.2, U3.3; no longer R13.1, U2.10
- net N$25: now also R15.1, U3.1; no longer C6.2, TR1.P$4
- net N$8: now also R13.1, R14.2, U3.4; no longer C31.2, U2.8
- net OUT_R: now also R14.1, U3.5; no longer U2.16
- net RF_2: now also TR1.P$4; no longer C6.1
- net VBAT: no longer C32.+, C33.2, U2.12, U2.13, U2.4, U2.5, U2.6
Routing:
- net VBAT: track 107.9 -> 54.0 mm, vias 2 -> 0
- net GND: track 448.4 -> 479.2 mm, vias 3 -> 6
- net RF_2: track 3.68 -> 21.9 mm
- net AGND: track 14.7 -> 0.00 mm, vias 2 -> 0
- net N$25: track 15.4 -> 2.40 mm
- net OUT_R: track 18.8 -> 27.4 mm
- net N$14: track 2.80 -> 11.3 mm
- net N$8: track 3.38 -> 11.2 mm
- net N$28: track 0.00 -> 6.61 mm
- net +3V3: track 195.3 -> 201.7 mm
- net N$29: track 0.00 -> 5.16 mm
- net N$2: track 35.2 -> 30.2 mm, vias 0 -> 2
- net D-: track 35.0 -> 37.1 mm
- net N$17: track 4.28 -> 2.36 mm
- net N$10: track 29.4 -> 31.0 mm
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Other:
- board text added: "Batt."
- board text added: "DL3AKB"
- board text added: "Headphones"
- board text added: "OLED"
- board text added: "PICO-SDR"
- board text added: "RF"
- board text added: "Sound-Card"
- board text added: "Speaker"
