File: 01_sheet/PICO_SDR.sch (EAGLE design)
At the start: 70 parts, among them IC2 MCP6022, J1 DCJ0202, J2 FC68131, J3 FC68133, SW1 EC12E_SW, U2 74CBTLV3253, U3 PAM8403DR

Commit message: sheet
Parts:
- added JP3: Speaker, pinhead:PINHD-1X2
- C11, C12, C13, C19, C2, C26, C27, C28, C29, C3, C6, C7: device rcl:C-EUC1206 -> rcl:C-EUC0805
- C14, C32: value (none) -> 100n
- C15, C16, C17, C20: value (none) -> 100µ; device rcl:CPOL-EUE2,5-6E -> rcl:CPOL-EUSMCD
- C18: value (none) -> 470n
- C21: value (none) -> 1µ
- C22: value (none) -> 470n; device rcl:C-EUC1206 -> rcl:C-EUC0805
- L1, L2: value (none) -> VK200
- R1: value (none) -> 100
- R2: value (none) -> 20k
- R3: value RK09K1130A6S -> 10k
Connections:
- new net N$26: C10.1, C12.2, L3.2
- new net N$27: C5.1, C6.2, L5.2
- net LP+: now also JP3.2
- net LP-: now also JP3.1
- net P_180: no longer C10.1, C12.2, L3.2
- net P_270: no longer C5.1, C6.2, L5.2

Commit message: new version
Parts:
- removed U$3: RP2350 - Stamp, rp2xxx_stamp:RP2040_STAMPTH
- removed U3: PAM8403DR, PAM8403DR:PAM8403DR
- added IC1: RP2350 - Stamp, rp2xxx_stamp:RP2040_STAMPSMD
- added J4: FC68133, FC68133:FC68133
- added JP4: RF, pinhead:PINHD-1X2
- added U1: 74CBTLV3253, FST3253MX:FST3253MX
- C1: value 220n -> 100n
- C10: value 10µ -> 10n; device rcl:C-EUC1206 -> rcl:C-EUC0805
- C13: value 100n -> 10n
- C14: value 100n -> 10n; device rcl:C-EUC1206 -> rcl:C-EUC0805
- C15, C16: value 100µ -> 10n; device rcl:CPOL-EUSMCD -> rcl:C-EUC0805
- C17, C20: value 100µ -> 10µ; device rcl:CPOL-EUSMCD -> rcl:C-EUC1206
- C18: value 470n -> 10µ
- C19: value 100n -> 10µ; device rcl:C-EUC0805 -> rcl:C-EUC1206
- C2: value 100n -> 100µ; device rcl:C-EUC0805 -> rcl:CPOL-EUSMCD
- C21: value 1µ -> 100µ; device rcl:C-EUC1206 -> rcl:CPOL-EUSMCD
- C22: device rcl:C-EUC0805 -> rcl:C-EUC1206
- C23: value 10µ -> 27p
- C26: value 10n -> 100n
- C27: value 10n -> 27p; device rcl:C-EUC0805 -> rcl:C-EUC1206
- C28, C29: value 10n -> 10µ; device rcl:C-EUC0805 -> rcl:C-EUC1206
- C3: value 2,2µ -> 100n; device rcl:C-EUC0805 -> rcl:C-EUC1206
- C30: value 10µ -> 470n; device rcl:C-EUC1206 -> rcl:C-EUC0805
- C31: value 10µ -> 100n; device rcl:C-EUC1206 -> rcl:C-EUC0805
- C32: value 100n -> 100µ; device rcl:C-EUC1206 -> rcl:CPOL-EUSMCD
- C33: value 220n -> 1µ
- C4: value 10µ -> 2,2µ; device rcl:C-EUC1206 -> rcl:C-EUC0805
- C5: value 10µ -> 220n
- C6: value 10n -> 220n; device rcl:C-EUC0805 -> rcl:C-EUC1206
- C7: value 10n -> 100µ; device rcl:C-EUC0805 -> rcl:CPOL-EUSMCD
- C8: value 27p -> 100n; device rcl:C-EUC1206 -> rcl:C-EUC0805
- C9: value 27p -> 10n; device rcl:C-EUC1206 -> rcl:C-EUC0805
- J2: value FC68131 -> 629105136821; device FC68131:FC68131 -> Eagle_WR-USB (rev25a):629105136821
- J3: value FC68133 -> FC68131; device FC68133:FC68133 -> FC68131:FC68131
- OLED1: value OLED -> (none)
- R1: value 100 -> 10k
- R12: value 100 -> 10k; device rcl:R-EU_R0805 -> RK09K1130A6S:RK09K1130A6S
- R13: value 100 -> 20k
- R2: value 20k -> 10k
- R3: value 10k -> 100; device RK09K1130A6S:RK09K1130A6S -> rcl:R-EU_R0805
- R4, R7: value 100k -> 100
- R5, R6: value 10k -> 100
- R8, R9: value 100 -> 100k
- U2: value 74CBTLV3253 -> PAM8403DR; device FST3253MX:FST3253MX -> PAM8403DR:PAM8403DR
- renumbered U$1 to TR1, U$2 to OLED1
Connections:
- new net D+: IC1.USB_D+, J2.D+
- new net D-: IC1.USB_D-, J2.D-
- net +3V3: now also C26.2, C3.2, C7.+, C8.1, R1.2, SJ1.2, SJ2.2, U1.VCC; no longer C13.2, C14.2, C16.+, C2.1, R6.2, SJ3.2, SJ4.2, U2.VCC
- net +5V: now also C1.2, C2.+, J2.VBUS; no longer C17.+, C32.2
- net AGND: now also C32.-, C33.1; no longer C20.-, C21.1
- net BAND_0: now also IC1.GPIO2; no longer U$3.GPIO2
- net BAND_1: now also IC1.GPIO3; no longer U$3.GPIO3
- net BAND_2: now also IC1.GPIO4; no longer U$3.GPIO4
- net BIAS: now also C27.2, C4.2, R1.1, R11.1, R2.2, R9.1; no longer C25.2, C3.2, R4.1, R5.2, R6.1, R7.1
- net BUTTON_BACK: now also IC1.GPIO17; no longer U$3.GPIO17
- net BUTTON_FWD: now also IC1.GPIO22; no longer U$3.GPIO22
- net CS: now also IC1.GPIO13; no longer U$3.GPIO13
- net ENCODER_A: now also IC1.GPIO21; no longer U$3.GPIO21
- net ENCODER_B: now also IC1.GPIO20; no longer U$3.GPIO20
- net GND: now also C1.1, C10.1, C15.1, C16.1, C2.-, C22.1, C31.1, C4.1, C7.-, C8.2, C9.1, IC1.GND, J2.GND, J2.SHIELD, J3.SLEEVE, R12.3, R2.1, SJ3.2, SJ4.2, U1.!OE!1, U1.!OE!2, U1.GND, U2.PGND@1, U2.PGND@2; no longer C16.-, C17.-, C18.1, C19.1, C2.2, C27.1, C28.1, C29.1, C32.1, C6.1, C7.1, J2.SLEEVE, R3.3, R5.1, SJ1.2, SJ2.2, U$3.GND, U2.!OE!1, U2.!OE!2, U3.GND, U3.PGND@1, U3.PGND@2
- net LO_I: now also IC1.GPIO1, U1.S1; no longer U$3.GPIO1, U2.S1
- net LO_Q: now also IC1.GPIO0, U1.S0; no longer U$3.GPIO0, U2.S0
- net LP+: now also J4.3, J4.4; no longer J3.3, J3.4
- net LP-: now also J4.1, U2.-OUT_R; no longer J3.1, U3.-OUT_R
- net MISO: now also IC1.GPIO12; no longer U$3.GPIO12
- net MOSI: now also IC1.GPIO15; no longer U$3.GPIO15
- net N$1: now also IC1.3.3V; no longer U$3.3.3V
- net N$10: now also C27.1, R11.2, R6.1; no longer C25.1, R7.2, R9.1
- net N$11: now also C25.1, R5.1; no longer C8.1, R8.1
- net N$12: now also C18.2, R4.2; no longer C4.2, R13.2
- net N$13: now also C23.1, R3.1, R8.2; no longer C9.1, R11.2, R12.1
- net N$14: now also R13.1, U2.INR; no longer R2.1, U3.INR
- net N$15: now also C17.2, R3.2; no longer C10.2, R12.2
- net N$16: now also R4.1, R9.2; no longer R13.1, R4.2
- net N$17: now also C30.1, R13.2; no longer C22.1, R2.2
- net N$18: now also C5.2; no longer C1.2
- net N$19: now also C20.2, R6.2; no longer C23.2, R9.2
- net N$2: now also C21.-, R7.2; no longer C15.-, R1.2
- net N$20: now also C15.2, C18.1; no longer C11.2, C4.1
- net N$21: now also C28.2, J3.TIP; no longer C30.2, J2.TIP
- net N$22: now also C29.2, J3.RING; no longer C31.2, J2.RING
- net N$23: now also SJ2.1, SJ4.1; no longer SJ1.1, SJ3.1
- net N$24: now also SJ1.1, SJ3.1; no longer SJ2.1, SJ4.1
- net N$25: now also C6.2; no longer C33.2
- net N$26: now also C13.2, C17.1; no longer C10.1, C12.2
- net N$27: now also C14.2, C19.1; no longer C5.1, C6.2
- net N$3: now also C16.2, C20.1; no longer C23.1, C7.2
- net N$4: now also IC1.5V; no longer U$3.5V
- net N$5: now also U1.2A; no longer U2.2A
- net N$6: now also C19.2, R5.2; no longer C5.2, R8.2
- net N$7: now also U1.1A; no longer U2.1A
- net N$8: now also C31.2, U2.VREF; no longer C19.2, U3.VREF
- net N$9: now also C30.2, R12.2; no longer C22.2, R3.2
- net NF: now also C22.2, R12.1, R7.1; no longer C18.2, R1.1, R3.1
- net OUT_R: now also J4.2, J4.5, U2.+OUT_R; no longer J3.2, J3.5, U3.+OUT_R
- net PUSH: now also IC1.GPIO5; no longer U$3.GPIO5
- net P_0: now also C11.2, U1.1B2, U1.2B3; no longer C26.2, U2.1B2, U2.2B3
- net P_180: now also C9.2, U1.1B3, U1.2B2; no longer C27.2, U2.1B3, U2.2B2
- net P_270: now also C10.2, U1.1B4, U1.2B1; no longer C29.2, U2.1B4, U2.2B1
- net P_90: now also C12.2, U1.1B1, U1.2B4; no longer C28.2, U2.1B1, U2.2B4
- net RF_1: now also C5.1, JP4.2; no longer C1.1
- net RF_2: now also C6.1, JP4.1; no longer C33.1
- net RX_I: now also C23.2, C28.1, IC1.GPIO27, R8.1; no longer C30.1, C9.2, R11.1, U$3.GPIO27
- net RX_Q: now also C25.2, C29.1, IC1.GPIO26; no longer C31.1, C8.2, U$3.GPIO26
- net SCK: now also IC1.GPIO14; no longer U$3.GPIO14
- net SCL: now also IC1.GPIO19; no longer U$3.GPIO19
- net SDA: now also IC1.GPIO18; no longer U$3.GPIO18
- net SPEAKER: now also C21.+, IC1.GPIO16; no longer C15.+, U$3.GPIO16
- net VBAT: now also C32.+, C33.2, IC1.VBAT, U2.MUTE, U2.PVDD@1, U2.PVDD@2, U2.SHND, U2.VDD; no longer C20.+, C21.2, U$3.VBAT, U3.MUTE, U3.PVDD@1, U3.PVDD@2, U3.SHND, U3.VDD
Other:
- moved on the sheet: C1, C10, C11, C12, C13, C14, C18, C19, C22, C23, C25, C26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

Commit message: new Version (08.07.25)
Parts:
- removed C32: 100µ, rcl:CPOL-EUSMCD
- removed J2: 629105136821, Eagle_WR-USB (rev25a):629105136821
- removed U2: PAM8403DR, PAM8403DR:PAM8403DR
- added FL1, FL2: BLM21SP111SH1D, BLM21SP111SH1D:BLM21SP111SH1D
- added J5: 629105150521, Eagle_WR-USB (rev25a):629105150521
- added R14: 40k, rcl:R-EU_R0805
- added R15: 20k, rcl:R-EU_R0805
- added U3: MAX9716EUAT, MAX9716EUAT:MAX9716EUAT
- C31: value 100n -> 1µ
- C6: value 220n -> 100n; device rcl:C-EUC1206 -> rcl:C-EUC0805
Connections:
- removed net AGND: C32.-, C33.1
- new net N$28: C6.1, FL1.1, SJ1.2, SJ2.2
- new net N$29: C8.1, FL2.2, U1.VCC
- net +3V3: now also C33.2, FL1.2, FL2.1, R15.2, U3.VCC; no longer C8.1, SJ1.2, SJ2.2, U1.VCC
- net +5V: now also J5.VBUS; no longer J2.VBUS
- net D+: now also J5.D+; no longer J2.D+
- net D-: now also J5.D-; no longer J2.D-
- net GND: now also C33.1, C6.2, J5.SHIELD, U3.EPAD, U3.GND; no longer J2.GND, J2.SHIELD, U2.GND, U2.PGND@1, U2.PGND@2
- net LP-: now also U3.OUT-; no longer U2.-OUT_R
- net N$14: now also C31.2, U3.BIAS, U3.IN+; no longer R13.1, U2.INR
- net N$25: now also R15.1, U3.!SHDN; no longer C6.2, TR1.P$2
- net N$8: now also R13.1, R14.2, U3.IN-; no longer C31.2, U2.VREF
- net OUT_R: now also R14.1, U3.OUT+; no longer U2.+OUT_R
- net RF_2: now also TR1.P$2; no longer C6.1
- net VBAT: no longer C32.+, C33.2, U2.MUTE, U2.PVDD@1, U2.PVDD@2, U2.SHND, U2.VDD
Other:
- moved on the sheet: C21, C22, C30, C31, C33, C6, C8, J4, JP3, R12, R13, R7
